File: Eagle/MazeSolverPCB.brd (EAGLE design)
At the start: 53.3 x 50.8 mm, 26 parts

Commit message: Fixed Resistor values and folder names
Parts:
- R1, R2, R3, R4: value (none) -> 470
- R5, R6: value (none) -> 220
- R7, R8: value (none) -> 10000
Connections:
- removed net N$16: X2.16
- removed net N$18: X3.10
- removed net N$22: X1.13
- removed net N$23: X3.11
- removed net N$24: D2.A, X3.1
- removed net N$31: X2.15
- new net N$15: D2.A, X3.1, X3.2
- net N$10: now also X2.2
- net N$20: now also X3.12
- net N$6: now also X2.4
- net N$8: now also X1.2
- net N$9: now also X2.3
Routing:
- net N$6: track 0.00 -> 61.8 mm
- net N$25: track 0.00 -> 45.2 mm
- net N$10: track 0.00 -> 34.2 mm
- net N$9: track 0.00 -> 29.8 mm
- net N$15: track 0.00 -> 25.8 mm
- net N$24: track 24.8 -> 0.00 mm
- net N$27: track 34.2 -> 46.9 mm
- net N$8: track 12.8 -> 15.1 mm
- net N$26: track 45.7 -> 44.4 mm
- net N$2: track 72.7 -> 73.3 mm
